Commit message: hw0

File: homework/hw0/rprbot.urdf (robot description, URDF)
Before this commit: robot rprbot, 4 links, 3 joints
Links:
- added link link3, mass 2; visual box size=0.1 0.15 0.05; visual cylinder length=2.5 radius=0.03
- link link1: geometry visual box size=0.1 0.15 0.05; visual cylinder length=2.5 radius=0.03
- link link2: mass 2 -> 0.01; geometry visual cylinder length=0.15 radius=0.06
Joints:
- added joint j3: type prismatic, parent link2, child link3, origin xyz=0 0 0 rpy=0 0 0, axis 0 0 1, limit lower=-2.967 upper=2.967 effort=176 velocity=1.7104
